File: schematics/Display/Display.kicad_sch (KiCad schematic)
At the start: 13 parts, among them M1 Stepper_Motor_unipolar_5pin, SW1 SW_SPST, U1 ESP32-WROOM-32, U2 SS1306, U3 ULN2003, U4 MT3608

Commit message: Update for PCB design review
Parts:
- removed BT1: Battery_Cell, symbol Device:Battery_Cell
- removed C1, C2: 22uF, symbol Device:C
- removed D1: SS34, Diode_SMD:D_SMA, symbol Diode:SS34
- removed L1: 22uH, symbol Device:L
- removed R1: 16k, symbol Device:R
- removed R2: 2.2k, symbol Device:R
- removed SW1: SW_SPST, symbol Switch:SW_SPST
- removed U1: ESP32-WROOM-32, RF_Module:ESP32-WROOM-32, symbol RF_Module:ESP32-WROOM-32
- removed U2: SS1306, symbol sensorcircuits:SSD1306_OLED
- removed U4: MT3608, Package_TO_SOT_SMD:SOT-23-6, symbol Regulator_Switching:MT3608
- added BT2: Battery_Cell, symbol Device:Battery_Cell
- added Brd1: SSD1306, symbol sensorcircuits:SSD1306
- added C3, C4: 22uF, symbol Device:C
- added D1, D2: WS2812B, LED_SMD:LED_WS2812B_PLCC4_5.0x5.0mm_P3.2mm, symbol LED:WS2812B
- added D3: SS34, Diode_SMD:D_SMA, symbol Diode:SS34
- added L2: 4.7uH, symbol Device:L
- added R3: 110k, symbol Device:R
- added R4: 15k, symbol Device:R
- added SW2: SW_SPST, symbol Switch:SW_SPST
- added U1: ~, symbol sensorcircuits:XIAO_ESP32
- added U5: MT3608, Package_TO_SOT_SMD:SOT-23-6, symbol Regulator_Switching:MT3608
Connections:
- net GND: now reaches U3.8 (GND)
- net GND: now also BT2.2 (-), Brd1.1 (GND), C3.2, C4.2, D1.3 (VSS), D2.3 (VSS), R4.1, U1.13 (GND), U1.16 (-BATT), U5.2 (GND)
- net IN1: now reaches U3.1 (IN1)
- net IN1: now also U1.1 (GPIO1_A0_D0)
- net IN2: now reaches U3.2 (IN2)
- net IN2: now also U1.2 (GPIO2_A1_D1)
- net IN3: now reaches U3.3 (IN3)
- net IN3: now also U1.3 (GPIO3_A2_D2)
- net IN4: now reaches U3.4 (IN4)
- net IN4: now also U1.4 (GPIO4_A3_D3)
- net +5V: now reaches M1.5, U3.9 (COM)
- net +5V: now also C4.1, D3.1 (K), R3.2
- new net: D3.2 (A), L2.2, U5.1 (SW)
- new net: D1.4 (DIN), U1.10 (GPIO8_A9_D9_CIPO)
- new net: BT2.1 (+), SW2.1 (A), U1.15 (+BATT)
- new net: D1.2 (DOUT), D2.4 (DIN)
- new net: C3.1, L2.1, SW2.2 (B), U5.4 (EN), U5.5 (IN)
- new net: R3.1, R4.2, U5.3 (FB)
- new net +3.3V: Brd1.2 (VCC), D1.1 (VDD), D2.1 (VDD), U1.12 (3V3)
- new net SCL: Brd1.3 (SCL), U1.6 (GPIO6_A5_D5_SCL)
- new net SDA: Brd1.4 (SDA), U1.5 (GPIO4_A3_D3_SDA)
Other:
- moved on the sheet: M1, U3
