File: schematics/Sensing/Sensing.kicad_pcb (KiCad board)
At the start: 2 copper layers, 91.9 x 23.9 mm, 15 parts, among them J1 Conn_01x02_Pin, J2 Conn_01x05_Pin, J3 Conn_01x05_Pin, SW1 SW_SPST, SW2 SW_Push, U2 TCS34725FN

Commit message: Custom PCB Design
Parts:
- U3: footprint ESP32_Xiao_Seeed:XIAO_ESP32 -> ESP32_Xiao_Seeed_GIX:XIAO_ESP32
- moved D3 4.94 mm to (70.8, 68.9)
- moved J2 4.94 mm to (80.5, 69.1)
- moved D1 4.94 mm to (70.8, 79.0)
- moved D4 4.94 mm to (75.4, 74.1)
- moved U2 4.94 mm to (70.7, 73.8)
- moved D2 4.94 mm to (65.5, 74.1)
Routing:
- net GND: track 120.0 -> 108.0 mm, vias 2 -> 1
- net Net-(SW1-B): track 23.5 -> 25.4 mm
- added copper zone on B.Cu, net GND
- added copper zone on F.Cu, net GND
Other:
- board size 91.9 x 23.9 mm -> 87 x 23.9 mm
- board text added: "Main Board"
- board text added: "Sensor Tip"
- board text added: "Two custom Split-PCB Design to manage the directional requirements of the sensor. The Main Board and Sensor Tip are linked via a flexible 1x5 Connector carrying 3.3V, GND, SDA, SCL, and LED Control."
- board text added: "Yutong Luo - Custom PCB Design for Sensing Device v1.0"
- board text added: "Yutong Luo v1.0"

Commit message: Update PCB and Enclosure Designs
Parts:
- removed D3, D4: LED, LED_SMD:LED_0603_1608Metric_Pad1.05x0.95mm_HandSolder
- removed J2, J3: Conn_01x05_Pin, Connector_PinSocket_2.54mm:PinSocket_1x05_P2.54mm_Vertical
- removed R3: 100, Resistor_SMD:R_0603_1608Metric_Pad0.98x0.95mm_HandSolder
- removed SW1: SW_SPST, Button_Switch_SMD:SW_SPST_EVQPE1
- removed SW2: SW_Push, Button_Switch_SMD:SW_SPDT_PCM12
- removed U2: TCS34725FN, TCS34725:TCS34725FN_AMS
- added C2: 1uF, Capacitor_SMD:C_0603_1608Metric_Pad1.08x0.95mm_HandSolder, F.Cu at (143.5, 89.3)
- added C3: 1uF, Capacitor_SMD:C_0603_1608Metric_Pad1.08x0.95mm_HandSolder, F.Cu at (135.6, 89.3)
- added Q1: BSS138, BSS138:SOT-23_3L_ONS, F.Cu at (135.3, 100.4)
- added Q2: BSS138, BSS138:SOT-23_3L_ONS, F.Cu at (143.3, 100.1)
- added R5: 4.7k, Resistor_SMD:R_0603_1608Metric_Pad0.98x0.95mm_HandSolder, F.Cu at (134.9, 94.8)
- added R6: 4.7k, Resistor_SMD:R_0603_1608Metric_Pad0.98x0.95mm_HandSolder, F.Cu at (131.6, 100.0)
- added R7: 4.7k, Resistor_SMD:R_0603_1608Metric_Pad0.98x0.95mm_HandSolder, F.Cu at (143.5, 94.8)
- added R8: 4.7k, Resistor_SMD:R_0603_1608Metric_Pad0.98x0.95mm_HandSolder, F.Cu at (146.8, 100.0)
- added U1: AS7341-DLGT, AS7341_DLGT:SON8_AS7341-DLGM_AMS, F.Cu at (138.6, 94.9)
- C1: footprint LED_SMD:LED_0603_1608Metric_Pad1.05x0.95mm_HandSolder -> Capacitor_SMD:C_0603_1608Metric_Pad1.08x0.95mm_HandSolder
- D1, D2: value LED -> MP-3030-120H-30-80; footprint LED_SMD:LED_0603_1608Metric_Pad1.05x0.95mm_HandSolder -> MP_3030_120H_30_80:LED_MP-3030-120H-30-80
- J1: value Conn_01x02_Pin -> Conn_01x04_Pin; footprint Connector_PinSocket_2.54mm:PinSocket_1x02_P2.54mm_Vertical -> Connector_PinSocket_2.54mm:PinSocket_1x04_P2.54mm_Vertical
- R1, R2: value 4.7k -> 22
- U3: value ~ -> MCP1700x-180xxTT; footprint ESP32_Xiao_Seeed_GIX:XIAO_ESP32 -> Package_TO_SOT_SMD:SOT-23
- moved D1 78.1 mm to (147.3, 94.7), turned to 180 degrees
- moved D2 68.7 mm to (131.0, 94.7), turned to 0 degrees
- moved J1 37.0 mm to (143.0, 104.4)
- moved R1 35.6 mm to (146.4, 90.2), turned to 0 degrees
- moved C1 29.0 mm to (139.2, 100.0), turned to 90 degrees
- moved R2 21.6 mm to (132.0, 90.2)
- moved U3 18.2 mm to (138.9, 89.2), turned to 180 degrees
Connections:
- C1 pad 1: +3.3V -> +1V8
- J1 pad 1: /+BATT -> +3.3V
- R1 pad 1: Net-(U3-GPIO4_A3_D3_SDA) -> /LDR
- R1 pad 2: /SDA -> Net-(D1-PadC)
- R2 pad 1: Net-(U3-GPIO6_A5_D5_SCL) -> /LDR
- R2 pad 2: /SCL -> Net-(D2-PadC)
- U3 pad 1: Net-(U3-GPIO1_A0_D0) -> GND
- U3 pad 2: Net-(U3-GPIO2_A1_D1) -> +1V8
- U3 pad 3: unconnected-(U3-GPIO3_A2_D2-Pad3) -> +3.3V
Routing:
- net GND: track 108.0 -> 35.6 mm, vias 1 -> 3
- net /SCL: track 41.0 -> 5.09 mm
- net /LED: track 31.4 -> 0.00 mm
- net /LDR: track 0.00 -> 26.5 mm
- net +3.3V: track 76.0 -> 50.0 mm, vias 1 -> 0
- net Net-(SW1-B): track 25.4 -> 0.00 mm
- net /SDA: track 28.8 -> 3.92 mm, vias 1 -> 0
- net +1V8: track 0.00 -> 23.1 mm, vias 0 -> 2
- net Net-(U3-GPIO1_A0_D0): track 17.6 -> 0.00 mm
- net /SCL_3V3: track 0.00 -> 10.6 mm
- net /+BATT: track 10.2 -> 0.00 mm
- net Net-(Q2-Pad2): track 0.00 -> 6.95 mm
- net Net-(U3-GPIO6_A5_D5_SCL): track 6.60 -> 0.00 mm
- net Net-(U3-GPIO4_A3_D3_SDA): track 6.56 -> 0.00 mm
- net Net-(U3-GPIO2_A1_D1): track 6.35 -> 0.00 mm
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Other:
- board size 87 x 23.9 mm -> 23 x 23 mm
- board text removed: "Main Board"
- board text removed: "Sensor Tip"
- board text removed: "Two custom Split-PCB Design to manage the directional requirements of the sensor. The Main Board and Sensor Tip are linked via a flexible 1x5 Connector carrying 3.3V, GND, SDA, SCL, and LED Control."
- board text removed: "Yutong Luo - Custom PCB Design for Sensing Device v1.0"
- board text removed: "Yutong Luo v1.0"
