File: schematics/Sensing/Sensing.kicad_sch (KiCad schematic)
At the start: 10 parts, among them SW1 SW_SPST, SW2 SW_Push, U1 MOUDLE-SEEEDUINO-XIAO-ESP32C3, U2 TCS34725FN

Commit message: Update for PCB design review
Parts:
- removed U1: MOUDLE-SEEEDUINO-XIAO-ESP32C3, MOUDLE14P-SMD-2.54-21X17.8MM, symbol LED:MOUDLE-SEEEDUINO-XIAO-ESP32C3
- added D2, D3, D4: LED, LED_SMD:LED_0603_1608Metric_Pad1.05x0.95mm_HandSolder, symbol Device:LED
- added J1: Conn_01x02_Pin, Connector_PinSocket_2.54mm:PinSocket_1x02_P2.54mm_Vertical, symbol Connector:Conn_01x02_Pin
- added J2, J3: Conn_01x05_Pin, Connector_PinSocket_2.54mm:PinSocket_1x05_P2.54mm_Vertical, symbol Connector:Conn_01x05_Pin
- added U3: ~, ESP32_Xiao_Seeed:XIAO_ESP32, symbol sensorcircuits:XIAO_ESP32
- C1, D1: footprint (none) -> LED_SMD:LED_0603_1608Metric_Pad1.05x0.95mm_HandSolder
- R1, R2, R3: footprint (none) -> Resistor_SMD:R_0603_1608Metric_Pad0.98x0.95mm_HandSolder
- SW1: footprint (none) -> Button_Switch_SMD:SW_SPST_EVQPE1
- SW2: footprint (none) -> Button_Switch_SMD:SW_SPDT_PCM12
- U2: footprint TCS34725FN_AMS -> TCS34725:TCS34725FN_AMS
Connections:
- net +3.3V: now reaches C1.1, U2.1 (VDD)
- net +3.3V: now also J2.1 (Pin_1), J3.1 (Pin_1), U3.12 (3V3); no longer R1.2, R2.2
- net at R2.1: now also U3.6 (GPIO6_A5_D5_SCL); no longer U2.2 (SCL)
- net GND: now reaches C1.2, U2.3 (GND)
- net GND: now also BT1.1 (+), SW2.2, D4.1 (K), J1.2 (Pin_2), J2.2 (Pin_2), J3.2 (Pin_2), U3.13 (GND), U3.16 (-BATT); no longer D1.1 (K), SW2.1
- net at R1.1: now also U3.5 (GPIO4_A3_D3_SDA); no longer U2.6 (SDA)
- net +BATT: now reaches SW1.1 (A)
- net +BATT: now also BT1.2 (-), J1.1 (Pin_1); no longer BT1.1 (+)
- net at SW1.2 (B): now also U3.15 (+BATT)
- net at R3.2: now also U3.2 (GPIO2_A1_D1)
- net LED: now reaches D1.2 (A), R3.1
- net LED: now also J2.5 (Pin_5), J3.5 (Pin_5)
- new net: D3.1 (K), D4.2 (A)
- new net: SW2.1, U3.1 (GPIO1_A0_D0)
- new net: D2.1 (K), D3.2 (A)
- new net: D1.1 (K), D2.2 (A)
- new net SCL: J2.4 (Pin_4), J3.4 (Pin_4), R2.2, U2.2 (SCL)
- new net SDA: J2.3 (Pin_3), J3.3 (Pin_3), R1.2, U2.6 (SDA)
Other:
- moved on the sheet: BT1, C1, D1, R1, R2, R3, SW1, SW2, U2

Commit message: Custom PCB Design
Parts:
- BT1: footprint (none) -> Xiao_Seeed_ESP32C3:MOUDLE14P-SMD-2.54-21X17.8MM
- C1: footprint LED_SMD:LED_0603_1608Metric_Pad1.05x0.95mm_HandSolder -> Capacitor_SMD:C_0603_1608Metric_Pad1.08x0.95mm_HandSolder
- U3: value ~ -> ESP32C3_Xiao; footprint ESP32_Xiao_Seeed:XIAO_ESP32 -> ESP32_Xiao_Seeed_GIX:XIAO_ESP32
Changed lines of the file:
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@@
 	(title_block
 		(title "Sensing Device (Pen)")
-		(date "2026-02-01")
+		(date "2026-02-04")
+		(rev "v2.0")
 	)
 	(junction
@@
 			)
 		)
-		(property "Footprint" ""
+		(property "Footprint" "Xiao_Seeed_ESP32C3:MOUDLE14P-SMD-2.54-21X17.8MM"
 			(at 252.476 109.22 90)
 			(effects
@@
 			)
 		)
-		(property "Value" "~"
+		(property "Value" "ESP32C3_Xiao"
 			(at 203.454 88.646 90)
 			(effects
@@
 			)
 		)
-		(property "Footprint" "ESP32_Xiao_Seeed:XIAO_ESP32"
+		(property "Footprint" "ESP32_Xiao_Seeed_GIX:XIAO_ESP32"
 			(at 207.01 86.36 0)
 			(effects
@@
 			)
 		)
-		(property "Footprint" "LED_SMD:LED_0603_1608Metric_Pad1.05x0.95mm_HandSolder"
+		(property "Footprint" "Capacitor_SMD:C_0603_1608Metric_Pad1.08x0.95mm_HandSolder"
 			(at 75.2348 99.06 0)
 			(effects

Commit message: Update PCB and Enclosure Designs
Parts:
- removed BT1: Battery_Cell, Xiao_Seeed_ESP32C3:MOUDLE14P-SMD-2.54-21X17.8MM, symbol Device:Battery_Cell
- removed D1, D2, D3, D4: LED, LED_SMD:LED_0603_1608Metric_Pad1.05x0.95mm_HandSolder, symbol Device:LED
- removed J1: Conn_01x02_Pin, Connector_PinSocket_2.54mm:PinSocket_1x02_P2.54mm_Vertical, symbol Connector:Conn_01x02_Pin
- removed J2, J3: Conn_01x05_Pin, Connector_PinSocket_2.54mm:PinSocket_1x05_P2.54mm_Vertical, symbol Connector:Conn_01x05_Pin
- removed R3: 100, Resistor_SMD:R_0603_1608Metric_Pad0.98x0.95mm_HandSolder, symbol Device:R
- removed SW1: SW_SPST, Button_Switch_SMD:SW_SPST_EVQPE1, symbol Switch:SW_SPST
- removed SW2: SW_Push, Button_Switch_SMD:SW_SPDT_PCM12, symbol Switch:SW_Push
- removed U2: TCS34725FN, TCS34725:TCS34725FN_AMS, symbol 2026-01-26_22-08-00:TCS34725FN
- removed U3: ESP32C3_Xiao, ESP32_Xiao_Seeed_GIX:XIAO_ESP32, symbol sensorcircuits:XIAO_ESP32
- added C2, C3: 1uF, Capacitor_SMD:C_0603_1608Metric_Pad1.08x0.95mm_HandSolder, symbol Device:C
- added D1, D2: MP-3030-120H-30-80, MP_3030_120H_30_80:LED_MP-3030-120H-30-80, symbol sensorcircuits:MP-3030-120H-30-80
- added J1: Conn_01x04_Pin, Connector_PinSocket_2.54mm:PinSocket_1x04_P2.54mm_Vertical, symbol Connector:Conn_01x04_Pin
- added Q1, Q2: BSS138, BSS138:SOT-23_3L_ONS, symbol sensorcircuits:BSS138
- added R5, R6, R7, R8: 4.7k, Resistor_SMD:R_0603_1608Metric_Pad0.98x0.95mm_HandSolder, symbol Device:R
- added U1: AS7341-DLGT, AS7341_DLGT:SON8_AS7341-DLGM_AMS, symbol sensorcircuits:AS7341-DLGT
- added U3: MCP1700x-180xxTT, Package_TO_SOT_SMD:SOT-23, symbol Regulator_Linear:MCP1700x-180xxTT
- R1, R2: value 4.7k -> 22
Connections:
- net +3.3V: now also C3.1, D1.A, D2.A, J1.1 (Pin_1), U3.3 (VI); no longer C1.1
- net GND: now also C2.2, C3.2, J1.2 (Pin_2), U1.3 (GND), U1.5 (PGND), U3.1 (GND)
- net SCL: now also R7.2, U1.2 (SCL); no longer R2.2
- net SDA: now also R5.2, U1.8 (SDA); no longer R1.2
- net LDR: now reaches R1.1
- net LDR: now also R2.1, U1.4 (LDR)
- new net: D1.C, R1.2
- new net: Q1.3, R6.2
- new net: Q1.2, R5.1
- new net: Q2.3, R8.2
- new net: Q2.2, R7.1
- new net: D2.C, R2.2
- new net +1V8: C1.1, C2.1, Q1.1, Q2.1, U1.1 (VDD), U3.2 (VO)
- new net SCL_3V3: J1.3 (Pin_3), R8.1
- new net SDA_3V3: J1.4 (Pin_4), R6.1
Other:
- title: Sensing Device (Pen) -> Sensing Device (Pen) - Sensor Tip
- moved on the sheet: C1
