File: schematics/Display_v2/Display_v2.kicad_pcb (KiCad board)
At the start: 2 copper layers, 90 x 50 mm, 9 parts, among them J1 Conn_01x02_Pin, J2 Conn_01x04_Pin, M1 Stepper_Motor_bipolar, SW2 SW_SPST

Commit message: Update code
Parts:
- removed Brd1: SSD1306, Display:Adafruit_SSD1306_No_Mounting_Holes
- removed D1, D2: WS2812B, LED_SMD:LED_WS2812B_PLCC4_5.0x5.0mm_P3.2mm
- removed SW2: SW_SPST, Button_Switch_SMD:SW_DIP_SPSTx01_Slide_6.7x4.1mm_W6.73mm_P2.54mm_LowProfile_JPin
- added J3: Conn_01x03_Pin, Connector_PinSocket_2.54mm:PinSocket_1x03_P2.54mm_Vertical, F.Cu at (211.3, 89.4)
- added J4: Conn_01x03_Pin, Connector_PinSocket_2.54mm:PinSocket_1x03_P2.54mm_Vertical, F.Cu at (231.1, 66.0)
- moved C3 3.05 mm to (231.1, 75.8)
Connections:
- C3 pad 1: Net-(SW2-B) -> Net-(J4-Pin_2)
- U1 pad 10: Net-(D1-DIN) -> /DI
- U1 pad 15: Net-(J1-Pin_2) -> Net-(J4-Pin_2)
Routing:
- net Net-(J1-Pin_2): track 78.6 -> 25.4 mm
- net Net-(J4-Pin_2): track 0.00 -> 46.1 mm
- net /DI: track 0.00 -> 45.4 mm
- net GND: track 100.5 -> 59.1 mm
- net Net-(D1-DIN): track 21.5 -> 0.00 mm
- net Net-(D1-DOUT): track 14.8 -> 0.00 mm
- net +3.3V: track 44.3 -> 30.8 mm
- net Net-(SW2-B): track 9.45 -> 0.00 mm
